Commit message: kinectic version

File: agvs_description/urdf/agvs.urdf.xacro (robot description, xacro)
@@ -114,5 +114,7 @@
   <transmission name="joint_bmw_trans">
 	 <type>transmission_interface/SimpleTransmission</type>
-     <joint name="joint_back_motor_wheel" />
+     <joint name="joint_back_motor_wheel">
+      <hardwareInterface>EffortJointInterface</hardwareInterface>
+    </joint>
      <actuator name="joint_bmw_motor">
 	    <hardwareInterface>EffortJointInterface</hardwareInterface>
@@ -153,8 +155,9 @@
   <transmission name="joint_bw_trans">
 	 <type>transmission_interface/SimpleTransmission</type>
-     <joint name="joint_back_wheel" />
+     <joint name="joint_back_wheel">
+	   <hardwareInterface>VelocityJointInterface</hardwareInterface>
+     </joint>
      <actuator name="joint_bw_motor">
 	   <!-- hardwareInterface>EffortJointInterface</hardwareInterface -->
-	   <hardwareInterface>VelocityJointInterface</hardwareInterface>
        <mechanicalReduction>${wheel_mechanical_reduction}</mechanicalReduction>
      </actuator>
@@ -193,7 +196,8 @@
   <transmission name="joint_fmw_trans">
 	 <type>transmission_interface/SimpleTransmission</type>
-     <joint name="joint_front_motor_wheel" />
+     <joint name="joint_front_motor_wheel">
+	    <hardwareInterface>EffortJointInterface</hardwareInterface>
+     </joint>
      <actuator name="joint_fmw_motor">
-	   <hardwareInterface>EffortJointInterface</hardwareInterface>
        <mechanicalReduction>${motor_wheel_mechanical_reduction}</mechanicalReduction>
        <!-- motorTorqueConstant>1</motorTorqueConstant -->
@@ -233,8 +237,8 @@
   <transmission name="joint_fw_trans">
 	 <type>transmission_interface/SimpleTransmission</type>
-     <joint name="joint_front_wheel" />
+     <joint name="joint_front_wheel">
+  	  <hardwareInterface>VelocityJointInterface</hardwareInterface>
+     </joint>
      <actuator name="joint_fw_motor">
-	   <!-- hardwareInterface>EffortJointInterface</hardwareInterface -->
-	   <hardwareInterface>VelocityJointInterface</hardwareInterface>
        <mechanicalReduction>${wheel_mechanical_reduction}</mechanicalReduction>
      </actuator>
@@ -273,7 +277,8 @@
   <transmission name="joint_swl_trans">
 	 <type>transmission_interface/SimpleTransmission</type>
-     <joint name="joint_side_wheel_left" />
+     <joint name="joint_side_wheel_left">
+	    <hardwareInterface>EffortJointInterface</hardwareInterface>
+     </joint>
      <actuator name="joint_swl_motor">
-	   <hardwareInterface>EffortJointInterface</hardwareInterface>
        <mechanicalReduction>${wheel_mechanical_reduction}</mechanicalReduction>
      </actuator>
@@ -312,7 +317,8 @@
   <transmission name="joint_swr_trans">
 	 <type>transmission_interface/SimpleTransmission</type>
-     <joint name="joint_side_wheel_right" />
+     <joint name="joint_side_wheel_right">
+	    <hardwareInterface>EffortJointInterface</hardwareInterface>
+     </joint>
      <actuator name="joint_swr_motor">
-	   <hardwareInterface>EffortJointInterface</hardwareInterface>
        <mechanicalReduction>${wheel_mechanical_reduction}</mechanicalReduction>
      </actuator>
@@ -347,7 +353,8 @@
   <transmission name="joint_elevator_trans">
 	 <type>transmission_interface/SimpleTransmission</type>
-     <joint name="elevator_joint" />
+     <joint name="elevator_joint">
+		  <hardwareInterface>EffortJointInterface</hardwareInterface>
+     </joint>
      <actuator name="elevator_motor">
-		<hardwareInterface>EffortJointInterface</hardwareInterface>
 		<mechanicalReduction>1000.0</mechanicalReduction>
 	 </actuator>
